File: KiCad/R1/DSMRlogger_v3_R1.sch (KiCad schematic (older format))
At the start: 17 parts, among them J1 RJ11-6, J2 Conn_02x04_Odd_Even, J3 Conn_01x01_Male, J4 Conn_01x01_Male, J5 Conn_01x01_Male, Q1 BC547, U1 MCP1700-3302E_TO92, U2 ESP-01v090

Commit message: Add PCB for through-hole
Parts:
- J1: footprint (none) -> Connectors-P1:RJ11-6
- J2: footprint (none) -> Pin_Headers:Pin_Header_Straight_2x04_Pitch2.54mm
- J3, J4, J5: footprint (none) -> Pin_Headers:Pin_Header_Straight_1x01_Pitch2.54mm
- R1, R2, R3, R4, R5, R6: footprint (none) -> Resistors_THT:R_Axial_DIN0207_L6.3mm_D2.5mm_P10.16mm_Horizontal
- U2: footprint (none) -> ESP8266:ESP-01
Changed lines of the file:
@@
 F 0 "J2" H 4425 2225 50  0000 C CNN
 F 1 "Conn_02x04_Odd_Even" H 4425 1725 50  0000 C CNN
-F 2 "" H 4375 2025 50  0001 C CNN
+F 2 "Pin_Headers:Pin_Header_Straight_2x04_Pitch2.54mm" H 4375 2025 50  0001 C CNN
 F 3 "" H 4375 2025 50  0001 C CNN
 	1    4375 2025
@@
 F 0 "J1" H 1975 2625 50  0000 C CNN
 F 1 "RJ11-6" H 1625 2625 50  0000 C CNN
-F 2 "" H 1775 2125 50  0001 C CNN
+F 2 "Connectors-P1:RJ11-6" H 1775 2125 50  0001 C CNN
 F 3 "" H 1775 2125 50  0001 C CNN
 	1    1775 2125
@@
 F 0 "U2" H 2750 4775 50  0000 C CNN
 F 1 "ESP-01v090" H 2750 4975 50  0000 C CNN
-F 2 "" H 2750 4875 50  0001 C CNN
+F 2 "ESP8266:ESP-01" H 2750 4875 50  0001 C CNN
 F 3 "" H 2750 4875 50  0001 C CNN
 	1    2750 4875
@@
 F 0 "R5" V 3955 4375 50  0000 C CNN
 F 1 "10k" V 3875 4375 50  0000 C CNN
-F 2 "" V 3805 4375 50  0001 C CNN
+F 2 "Resistors_THT:R_Axial_DIN0207_L6.3mm_D2.5mm_P10.16mm_Horizontal" V 3805 4375 50  0001 C CNN
 F 3 "" H 3875 4375 50  0001 C CNN
 	1    3875 4375
@@
 F 0 "R6" V 4330 4375 50  0000 C CNN
 F 1 "10k" V 4250 4375 50  0000 C CNN
-F 2 "" V 4180 4375 50  0001 C CNN
+F 2 "Resistors_THT:R_Axial_DIN0207_L6.3mm_D2.5mm_P10.16mm_Horizontal" V 4180 4375 50  0001 C CNN
 F 3 "" H 4250 4375 50  0001 C CNN
 	1    4250 4375
@@
 F 0 "R4" V 1580 4375 50  0000 C CNN
 F 1 "10k" V 1500 4375 50  0000 C CNN
-F 2 "" V 1430 4375 50  0001 C CNN
+F 2 "Resistors_THT:R_Axial_DIN0207_L6.3mm_D2.5mm_P10.16mm_Horizontal" V 1430 4375 50  0001 C CNN
 F 3 "" H 1500 4375 50  0001 C CNN
 	1    1500 4375
@@
 F 0 "R3" V 8230 4325 50  0000 C CNN
 F 1 "2.2k" V 8150 4325 50  0000 C CNN
-F 2 "" V 8080 4325 50  0001 C CNN
+F 2 "Resistors_THT:R_Axial_DIN0207_L6.3mm_D2.5mm_P10.16mm_Horizontal" V 8080 4325 50  0001 C CNN
 F 3 "" H 8150 4325 50  0001 C CNN
 	1    8150 4325
@@
 F 0 "R1" V 7580 4875 50  0000 C CNN
 F 1 "1k" V 7500 4875 50  0000 C CNN
-F 2 "" V 7430 4875 50  0001 C CNN
+F 2 "Resistors_THT:R_Axial_DIN0207_L6.3mm_D2.5mm_P10.16mm_Horizontal" V 7430 4875 50  0001 C CNN
 F 3 "" H 7500 4875 50  0001 C CNN
 	1    7500 4875
@@
 F 0 "R2" V 7280 4550 50  0000 C CNN
 F 1 "2.2k" V 7200 4550 50  0000 C CNN
-F 2 "" V 7130 4550 50  0001 C CNN
+F 2 "Resistors_THT:R_Axial_DIN0207_L6.3mm_D2.5mm_P10.16mm_Horizontal" V 7130 4550 50  0001 C CNN
 F 3 "" H 7200 4550 50  0001 C CNN
 	1    7200 4550
@@
 F 0 "J3" H 4275 2700 50  0000 C CNN
 F 1 "Conn_01x01_Male" H 4275 2500 50  0000 C CNN
-F 2 "" H 4275 2600 50  0001 C CNN
+F 2 "Pin_Headers:Pin_Header_Straight_1x01_Pitch2.54mm" H 4275 2600 50  0001 C CNN
 F 3 "" H 4275 2600 50  0001 C CNN
 	1    4275 2600
@@
 F 0 "J4" H 4275 3050 50  0000 C CNN
 F 1 "Conn_01x01_Male" H 4275 2850 50  0000 C CNN
-F 2 "" H 4275 2950 50  0001 C CNN
+F 2 "Pin_Headers:Pin_Header_Straight_1x01_Pitch2.54mm" H 4275 2950 50  0001 C CNN
 F 3 "" H 4275 2950 50  0001 C CNN
 	1    4275 2950
@@
 F 0 "J5" H 4275 3325 50  0000 C CNN
 F 1 "Conn_01x01_Male" H 4275 3125 50  0000 C CNN
-F 2 "" H 4275 3225 50  0001 C CNN
+F 2 "Pin_Headers:Pin_Header_Straight_1x01_Pitch2.54mm" H 4275 3225 50  0001 C CNN
 F 3 "" H 4275 3225 50  0001 C CNN
 	1    4275 3225
